Commit message: Update robot_core.xacro

File: description/robot_core.xacro (robot description, xacro)
@@ -4,5 +4,5 @@
     <xacro:property name="chassis_radius" value="0.125"/>
     <xacro:property name="chassis_thickness" value="0.125"/>
-    <xacro:property name="chassis_mass" value="1.5"/>
+    <xacro:property name="chassis_mass" value="2.5"/>
     <xacro:property name="wheel_radius" value="0.0325"/>
     <xacro:property name="wheel_thickness" value="0.025"/>
