Commit message: More Changes

File: description/gazebo_control.xacro (robot description, xacro)
@@ -6,5 +6,5 @@
             <left_joint>left_wheel_joint</left_joint>
             <right_joint>right_wheel_joint</right_joint>
-            <wheel_separation>0.150</wheel_separation>
+            <wheel_separation>0.180</wheel_separation>
             <wheel_diameter>0.066</wheel_diameter>
             <!-- Limits -->

File: description/robot_core.xacro (robot description, xacro)
@@ -9,5 +9,5 @@
     <xacro:property name="wheel_mass" value="0.05"/>
     <xacro:property name="wheel_offset_x" value="0.06"/>
-    <xacro:property name="wheel_offset_y" value="0.075"/>
+    <xacro:property name="wheel_offset_y" value="0.09"/>
     <xacro:property name="wheel_offset_z" value="0.0"/>
     <xacro:property name="caster_wheel_A_radius" value="0.0225"/>
